File: KiCAD/MiniVCF 1.1/MiniVCF.kicad_pcb (KiCad board)
At the start: 2 copper layers, 94 x 128.5 mm, 86 parts, among them J1 JST_BUS, J10 CV2, J11 CTRL_PANEL_CONN2, J12 MAIN_BOARD_CONN2, J2 IDC_BUS, J3 AudioIn, J4 CV1, J5 AudioOut, J6 CONN_PWR1, J7 CONN_PWR2, J8 MAIN_BOARD_CONN, J9 CTRL_PANEL_CONN, U1 TL074, U2 TL074

Commit message: Added v1.1 with initial fixes
Parts:
- moved D12 27.0 mm to (88.5, 83.8)
- moved D13 27.0 mm to (95.0, 83.8)
- moved D14 27.0 mm to (92.0, 56.5)
- moved D15 27.0 mm to (98.5, 56.5)
- moved D11 1.85 mm to (126.9, 125.1)
- moved R16 1.85 mm to (132.2, 132.7)
- moved D10 1.85 mm to (129.4, 132.7)
Connections:
- CUTOFF1 pad 1: POS12V_1 -> NEG12V_1
- CUTOFF1 pad 3: NEG12V_1 -> POS12V_1
- POST_LPF1 pad 1: A_AUDIO_OUT -> Net-(C14-Pad2)
- POST_LPF1 pad 3: Net-(C14-Pad2) -> A_AUDIO_OUT
Routing:
- net Net-(D10-Pad2): track 34.0 -> 20.6 mm
- net RESO_FEEDBACK: track 55.2 -> 48.4 mm
- net POS12V_1: track 88.5 -> 94.3 mm
- net A_AUDIO_OUT: track 34.2 -> 36.5 mm
- net Net-(CV_AMT1-Pad3): track 20.9 -> 22.6 mm
- net NEG12V_1: track 5.04 -> 3.86 mm
- net Net-(C14-Pad2): track 67.0 -> 68.0 mm
- net A_CLIPPING_LEDS: track 43.3 -> 43.9 mm
- net GND2: vias 87 -> 83
- net GND1: vias 92 -> 82

Commit message: Updated version number
Other:
- board text added: "MiniVCF v1.1"
Changed lines of the file:
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@@
     (effects (font (size 1 1) (thickness 0.15)))
   )
-  (gr_text "MiniVCF v1.0" (at 93.6 63.1) (layer F.SilkS)
+  (gr_text "MiniVCF v1.1" (at 93.6 63.1) (layer F.SilkS)
     (effects (font (size 1 1) (thickness 0.15)))
   )
