File: KiCAD/MiniVCF 1.1/MiniVCF.kicad_pcb (KiCad board)
At the start: 2 copper layers, 94 x 128.5 mm, 86 parts, among them J1 JST_BUS, J10 CV2, J11 CTRL_PANEL_CONN2, J12 MAIN_BOARD_CONN2, J2 IDC_BUS, J3 AudioIn, J4 CV1, J5 AudioOut, J6 CONN_PWR1, J7 CONN_PWR2, J8 MAIN_BOARD_CONN, J9 CTRL_PANEL_CONN, U1 TL074, U2 TL074

Commit message: Added files for v1.1
Parts:
- moved D11 3.06 mm to (126.3, 122.1)
- moved D10 3.06 mm to (128.8, 129.7)
- moved R16 3.06 mm to (131.6, 129.7)
Routing:
- net Net-(D10-Pad2): track 20.6 -> 34.4 mm
- net RESO_FEEDBACK: track 48.4 -> 55.1 mm
- net GND2: vias 81 -> 80
